File: fortuna-s/untitled.kicad_sch (KiCad schematic)
At the start: 5 parts

Commit message: .
Parts:
- removed U?: 74HC74, symbol 74xx:74HC74
- added U?: 74HC595, symbol 74xx:74HC595
- added U?: 74HC165, symbol 74xx:74HC165
Connections:
- net D0: no longer J?.2 (SCK)
- net D1: no longer J?.3 (MOSI)
- net GND: now also U?.10 (DS), U?.15 (~{CE}), U?.8 (GND), U?.8 (GND)
- net VCC: now also U?.16 (VCC), U?.16 (VCC)
- net ~{RD_SD}: now also U?.13 (~{OE})
- net ~{WR_SD}: now also U?.1 (~{PL}); no longer J?.1 (CS)
- new net: J?.3 (MOSI), U?.9 (Q7)
- new net ???: U?.2 (CP)
- no-connect marks 6 -> 7
