File: fortuna-s/fortuna-s.kicad_sch (KiCad schematic)
At the start: 4 parts

Commit message: .
Parts:
- added C? (x2): 22p, symbol Device:C
- added C?: 1uF, symbol Device:C
- added D?: 1N4148, Diode_THT:D_DO-35_SOD27_P7.62mm_Horizontal, symbol Diode:1N4148
- added D?: GREEN, symbol Device:LED
- added P?: USB_C_Plug_USB2.0, symbol Connector:USB_C_Plug_USB2.0
- added R? (x4): 10K, symbol Device:R_US
- added R? (x2): 100, symbol Device:R_US
- added R? (x2): 1K, symbol Device:R_US
- added R?: 1M, symbol Device:R_US
- added SW?: RESET, symbol Switch:SW_Push
- added SW?: POWER, symbol Switch:SW_DIP_x02
- added U? (x2): 74HCT04, symbol 74xx:74HCT04
- added U?: Z80CPU, symbol CPU:Z80CPU
- added Y?: 7.3728Mhz, symbol Device:Crystal
- J?: value FTDI -> FTDI cable
Connections:
- net CLK: now also U?.6, U?.6 (~{CLK})
- net GND: now also C?.2, C?.2, C?.2, P?.A1 (GND), P?.A12 (GND), P?.B1 (GND), P?.B12 (GND), R?.2, SW?.1, U?.29 (GND)
- net ~{INT}: now also R?.1, U?.16 (~{INT})
- net ~{M1}: now also U?.27 (~{M1})
- net +5V renamed VCC
- net VCC: now also D?.1 (K), D?.2 (A), R?.2, R?.2, R?.2, R?.2, R?.2, SW?.2, SW?.3, SW?.4, U?.11 (VCC)
- net WR renamed ~{WR}
- net ~{WR}: now also U?.22 (~{WR})
- new net: R?.2, SW?.2
- new net: C?.1, R?.1, U?.3, Y?.1
- new net: C?.1, R?.1, Y?.2
- new net: D?.1 (K), R?.1
- new net: P?.A4 (VBUS), P?.A9 (VBUS), P?.B4 (VBUS), P?.B9 (VBUS), SW?.1
- new net: R?.2, R?.2, U?.4, U?.5
- new net ~{BUSACK}: U?.23 (~{BUSACK})
- new net ~{BUSRQ}: R?.1, U?.25 (~{BUSRQ})
- new net ~{HALT}: U?.18 (~{HALT})
- new net ~{IORQ}: U?.20 (~{IORQ})
- new net ~{MREQ}: U?.19 (~{MREQ})
- new net ~{NMI}: R?.1, U?.17 (~{NMI})
- new net ~{RD}: U?.21 (~{RD})
- new net ~{RST}: C?.1, D?.2 (A), R?.1, R?.1, U?.26 (~{RESET})
- new net ~{WAIT}: R?.1, U?.24 (~{WAIT})
- no-connect marks 1 -> 7
Other:
- note added: "CLOCK"
- note added: "MICROPROCESSOR"
- note added: "Occupies 0x80 to 0xBF in memory map."
- note added: "POWER"
- note added: "RESET"
- note added: "The computer can be powered by the FTDI cable, but current can't exceed 350 mA."
- note added: "UART"
- note removed: "7.3728Mhz"
- note removed: "FTDI with the 5V jumper Whole circuit current should not exceed 350mA."
- note removed: "Occupies 0x80 to 0xBF."
- note removed: "POWER & UART"
- note removed: "USB cable ->"
- moved on the sheet: J?, R?, U?, U?A

Commit message: .
Parts:
- added J?: Ext Pinout, symbol Connector_Generic:Conn_02x10_Counter_Clockwise
- added R? (x4): 10K, symbol Device:R_US
- added U? (x4): 74LS32, symbol 74xx:74LS32
- added U?: 28C256, symbol Memory_EEPROM:28C256
- added U?: AS6C4008-55PCN, Package_DIP:DIP-32_W15.24mm, symbol Memory_RAM:AS6C4008-55PCN
- added U?: 74HCT04, symbol 74xx:74HCT04
Connections:
- net ~{IRQ} is gone; now on net ~{IORQ}: U?.1
- net A0: now also J?.20 (Pin_20)
- net A7: now also J?.18 (Pin_18)
- net GND: now also J?.10 (Pin_10), R?.1, R?.1, R?.1, U?.1 (A14), U?.14 (GND), U?.16 (VSS), U?.26 (A13)
- net VCC: now also J?.1 (Pin_1), R?.2, U?.28 (VCC), U?.32 (VCC)
- net ~{INT}: now also J?.14 (Pin_14)
- net ~{IORQ}: now also J?.17 (Pin_17)
- net ~{M1}: now also J?.15 (Pin_15)
- net ~{MREQ}: now also U?.2, U?.4
- net ~{RD}: now also U?.1
- net ~{WAIT}: now also J?.13 (Pin_13)
- net ~{WR}: now also J?.16 (Pin_16), U?.5
- net at U?.3 (A13): now also U?.10
- net at U?.4 (A14): now also U?.9
- net at U?.5 (A15): now also U?.12
- net ~{HALT}: no longer names the net of U?.18 (~{HALT})
- new net: U?.13, U?.8
- new net: U?.22 (~{OE}), U?.24 (OE#), U?.3
- new net: U?.22 (CE#), U?.8
- new net: U?.29 (WE#), U?.6
- new net A1: J?.19 (Pin_19)
- new net A13: U?.28 (A13)
- new net A14: U?.3 (A14)
- new net A15: U?.31 (A15)
- new net A16: R?.2, U?.2 (A16)
- new net A17: R?.2, U?.30 (A17)
- new net A18: R?.2, U?.1 (A18)
- new net ~{BOTTOM 8K}: U?.11, U?.20 (~{CS}), U?.9
- new net ~{ROM WE}: R?.1, U?.27 (~{WE})
- no-connect marks 7 -> 10
Other:
- note added: "EXTERNAL PORTS"
- note added: "MEMORY"
- moved on the sheet: C?, D?, J?, P?, R?, SW?, U?, U?A, U?B, U?C, Y?

Commit message: .
Parts:
- added J?: Debugger Pinout, symbol Connector_Generic:Conn_02x20_Counter_Clockwise
- added JP?: Clock, symbol Jumper:Jumper_2_Open
Connections:
- net A14: now also J?.27 (Pin_27)
- net A15: now also J?.26 (Pin_26)
- net A16: now also J?.25 (Pin_25)
- net A17: now also J?.24 (Pin_24)
- net A18: now also J?.23 (Pin_23)
- net CLK: now also J?.21 (Pin_21), JP?.2 (B); no longer U?.6
- net GND: now also J?.20 (Pin_20)
- net VCC: now also J?.1 (Pin_1)
- net ~{BUSACK}: now also J?.17 (Pin_17)
- net ~{BUSRQ}: now also J?.16 (Pin_16)
- net ~{INT}: now also J?.10 (Pin_10)
- net ~{IORQ}: now also J?.15 (Pin_15)
- net ~{M1}: now also J?.22 (Pin_22)
- net ~{MREQ}: now also J?.14 (Pin_14)
- net ~{RD}: now also J?.12 (Pin_12)
- net ~{ROM WE}: now also J?.18 (Pin_18)
- net ~{WAIT}: now also J?.11 (Pin_11)
- net ~{WR}: now also J?.13 (Pin_13)
- net ~{NMI}: no longer names the net of R?.1, U?.17 (~{NMI})
- new net: JP?.1 (A), U?.6
- no-connect marks 10 -> 11
Other:
- note added: "DEBUGGER"
- moved on the sheet: C?, D?, J?, R?, SW?, U?, U?A, U?B, U?C, U?D

Commit message: .
Connections:
- net RX: now also J?.12 (Pin_12)
- net TX: now also J?.11 (Pin_11)
- no-connect marks 11 -> 9
Other:
- note added: "Board: 55x37"
Changed lines of the file:
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@@
   (junction (at 217.17 97.79) (diameter 0) (color 0 0 0 0)
   )
-  (no_connect (at 261.62 209.55))
-  (no_connect (at 261.62 207.01))
   (no_connect (at 63.5 233.68))
   (no_connect (at 63.5 228.6))
@@
     (stroke (width 0) (type default) (color 0 0 0 0))
   )
+  (wire (pts (xy 261.62 209.55) (xy 270.51 209.55))
+    (stroke (width 0) (type default) (color 0 0 0 0))
+  )
   (wire (pts (xy 217.17 80.01) (xy 217.17 83.82))
     (stroke (width 0) (type default) (color 0 0 0 0))
@@
   )
   (wire (pts (xy 36.83 208.28) (xy 36.83 215.9))
+    (stroke (width 0) (type default) (color 0 0 0 0))
+  )
+  (wire (pts (xy 261.62 207.01) (xy 270.51 207.01))
     (stroke (width 0) (type default) (color 0 0 0 0))
   )
@@
     (effects (font (size 1.27 1.27) italic) (justify left bottom))
   )
+  (text "Board: 55x37" (at 405.13 250.19 180)
+    (effects (font (size 1.27 1.27)) (justify right bottom))
+  )
   (text "MICROPROCESSOR" (at 48.26 177.8 0)
     (effects (font (size 3 3) (thickness 0.6) bold) (justify left bottom))
@@
     (effects (font (size 1.27 1.27)) (justify left bottom))
   )
+  (label "TX" (at 270.51 209.55 180)
+    (effects (font (size 1.27 1.27)) (justify right bottom))
+  )
   (label "A7" (at 270.51 191.77 180)
     (effects (font (size 1.27 1.27)) (justify right bottom))
@@
     (effects (font (size 1.27 1.27)) (justify left bottom))
   )
+  (label "RX" (at 270.51 207.01 180)
+    (effects (font (size 1.27 1.27)) (justify right bottom))
+  )
   (symbol (lib_id "Device:R_US") (at 36.83 204.47 180) (unit 1)

Commit message: .
Parts:
- removed J?: Ext Pinout, symbol Connector_Generic:Conn_02x10_Counter_Clockwise
- added J?: Ext Pinout, symbol Connector_Generic:Conn_02x13_Counter_Clockwise
Connections:
- net A0: now also J?.26 (Pin_26)
- net A1: now also J?.25 (Pin_25)
- net A16: now also J?.10 (Pin_10)
- net A17: now also J?.11 (Pin_11)
- net A18: now also J?.12 (Pin_12)
- net A7: now also J?.24 (Pin_24)
- net GND: now also J?.13 (Pin_13)
- net RX: now also J?.18 (Pin_18)
- net TX: now also J?.17 (Pin_17)
- net VCC: now also J?.1 (Pin_1)
- net ~{INT}: now also J?.20 (Pin_20)
- net ~{IORQ}: now also J?.23 (Pin_23)
- net ~{M1}: now also J?.21 (Pin_21)
- net ~{WAIT}: now also J?.19 (Pin_19)
- net ~{WR}: now also J?.22 (Pin_22)
- net ~{NMI}: now reaches R?.1, U?.17 (~{NMI})
- net ~{NMI}: now also J?.19 (Pin_19)
- new net RST: J?.16 (Pin_16)
- no-connect marks 9 -> 8
Other:
- added sheet External board (untitled.kicad_sch)

Commit message: .
Parts:
- removed C? (x2): 22p, symbol Device:C
- removed R?: 1K, symbol Device:R_US
- removed R?: 1M, symbol Device:R_US
- removed U? (x2): 74HCT04, symbol 74xx:74HCT04
- removed Y?: 7.3728Mhz, symbol Device:Crystal
- added C? (x4): 10uF, symbol Device:C
- added X?: 7.3728 MHz, Oscillator:Oscillator_DIP-14, symbol Oscillator:ACO-xxxMHz
Connections:
- net A13: now also J?.27 (Pin_27)
- net A14: now also J?.26 (Pin_26); no longer J?.27 (Pin_27)
- net A15: now also J?.25 (Pin_25); no longer J?.26 (Pin_26)
- net A16: no longer J?.25 (Pin_25)
- net A17: no longer J?.24 (Pin_24)
- net A18: no longer J?.23 (Pin_23)
- net CLK: now also J?.22 (Pin_22); no longer J?.21 (Pin_21)
- net GND: now also J?.19 (Pin_19), C?.2, C?.2, C?.2, C?.2, X?.7 (GND); no longer J?.20 (Pin_20)
- net VCC: now also C?.1, C?.1, C?.1, C?.1, X?.14 (Vcc)
- net ~{M1}: now also J?.23 (Pin_23); no longer J?.22 (Pin_22)
- net ~{NMI}: now also J?.24 (Pin_24); no longer J?.19 (Pin_19)
- net at JP?.1 (A): now also X?.8 (OUT)
Other:
- note added: "TODO: add debugger using MEGA 2560 around Z80"
- note added: "Two hole internal spacing."
- moved on the sheet: J?, JP?

Commit message: .
Parts:
- removed J?: Debugger Pinout, symbol Connector_Generic:Conn_02x20_Counter_Clockwise
- removed J?: Ext Pinout, symbol Connector_Generic:Conn_02x13_Counter_Clockwise
- added C1, C2: 10uF, symbol Device:C
- added J1: Ext Pinout, symbol Connector_Generic:Conn_02x13_Counter_Clockwise
- added J2, J3: Conn_01x21, symbol Connector_Generic:Conn_01x21
- added U1: 74HTC138, symbol 74xx:74LS138
- added U2: 74HTC175, symbol 74xx:74LS175
Connections:
- net A0: now also J3.12 (Pin_12), U1.2 (A1)
- net A1: now also J3.11 (Pin_11), U1.3 (A2)
- net A13: now also J2.4 (Pin_4)
- net A14: now also J2.5 (Pin_5)
- net A15: now also J2.6 (Pin_6)
- net A16: now also J2.19 (Pin_19), U2.2 (Q0)
- net A17: now also J3.14 (Pin_14), U2.7 (Q1)
- net A18: now also J3.18 (Pin_18), U2.10 (Q2)
- net A6: now also J3.6 (Pin_6)
- net A7: now also J3.5 (Pin_5), U1.4 (E1)
- net CLK: now also J2.7 (Pin_7)
- net GND: now also C1.2, C2.2, J1.13 (Pin_13), J3.13 (Pin_13), U1.8 (GND), U2.13 (D3), U2.8 (GND)
- net RST: now also J1.22 (Pin_22), U2.1 (~{Mr})
- net RX: now also J1.24 (Pin_24)
- net TX: now also J1.23 (Pin_23)
- net VCC: now also C1.1, C2.1, J1.1 (Pin_1), J2.12 (Pin_12), U1.16 (VCC), U2.16 (VCC)
- net ~{BUSRQ}: now also J3.17 (Pin_17)
- net ~{INT}: now also J1.26 (Pin_26), J2.17 (Pin_17)
- net ~{IORQ}: now also J2.21 (Pin_21), U1.5 (E2)
- net ~{M1}: now also J3.15 (Pin_15), U1.6 (E3)
- net ~{MREQ}: now also J2.20 (Pin_20)
- net ~{NMI}: now also J2.18 (Pin_18)
- net ~{RD}: now also J3.21 (Pin_21)
- net ~{RST}: now also J3.16 (Pin_16)
- net ~{WAIT}: now also J1.25 (Pin_25)
- net ~{WR}: now also J3.20 (Pin_20)
- new net: U1.14 (O1), U2.9 (Cp)
- new net A10: J3.2 (Pin_2)
- new net A11: J2.2 (Pin_2)
- new net A12: J2.3 (Pin_3)
- new net A2: J1.21 (Pin_21), J3.10 (Pin_10)
- new net A3: J1.20 (Pin_20), J3.9 (Pin_9)
- new net A4: J3.8 (Pin_8)
- new net A5: J3.7 (Pin_7)
- new net A8: J3.4 (Pin_4)
- new net A9: J3.3 (Pin_3)
- new net D0: J2.15 (Pin_15), U2.4 (D0)
- new net D1: J2.16 (Pin_16), U2.5 (D1)
- new net D2: J2.13 (Pin_13), U2.12 (D2)
- new net D3: J2.9 (Pin_9)
- new net D4: J2.8 (Pin_8)
- new net D5: J2.10 (Pin_10)
- new net D6: J2.11 (Pin_11)
- new net D7: J2.14 (Pin_14)
- new net WR: U1.1 (A0)
- new net ~{BUSAK}: J3.19 (Pin_19)
- new net ~{ROM_WE}: J3.1 (Pin_1)
- new net ~{Y1R}: J1.19 (Pin_19), U1.13 (O2)
- new net ~{Y1W}: J1.18 (Pin_18), U1.12 (O3)
- new net ~{Y2R}: J1.17 (Pin_17), U1.11 (O4)
- new net ~{Y2W}: J1.16 (Pin_16), U1.10 (O5)
- new net ~{Y3R}: J1.15 (Pin_15), U1.9 (O6)
- new net ~{Y3W}: J1.14 (Pin_14), U1.7 (O7)
- no-connect marks 8 -> 18
Other:
- removed sheet External board
- note added: "BANKSWITCHING"
- note added: "EXTERNAL I/O"
- note added: "I/O MULTIPLEXER"
- note added: "IO address: write to 0x0"
- note removed: "EXTERNAL PORTS"
- note removed: "TODO: add debugger using MEGA 2560 around Z80"
- note removed: "Two hole internal spacing."
- moved on the sheet: C?

Commit message: .
Connections:
- net A0: now also J3.11 (Pin_11); no longer J3.12 (Pin_12)
- net A1: now also J3.10 (Pin_10); no longer J3.11 (Pin_11)
- net A10: now also J3.1 (Pin_1); no longer J3.2 (Pin_2)
- net A11: now also J2.1 (Pin_1); no longer J2.2 (Pin_2)
- net A12: now also J2.2 (Pin_2); no longer J2.3 (Pin_3)
- net A13: now also J2.3 (Pin_3); no longer J2.4 (Pin_4)
- net A14: now also J2.4 (Pin_4); no longer J2.5 (Pin_5)
- net A15: now also J2.5 (Pin_5); no longer J2.6 (Pin_6)
- net A16: now also J2.18 (Pin_18); no longer J2.19 (Pin_19)
- net A17: now also J3.13 (Pin_13); no longer J3.14 (Pin_14)
- net A18: now also J3.17 (Pin_17); no longer J3.18 (Pin_18)
- net A2: now also J3.9 (Pin_9); no longer J3.10 (Pin_10)
- net A3: now also J3.8 (Pin_8); no longer J3.9 (Pin_9)
- net A4: now also J3.7 (Pin_7); no longer J3.8 (Pin_8)
- net A5: now also J3.6 (Pin_6); no longer J3.7 (Pin_7)
- net A6: now also J3.5 (Pin_5); no longer J3.6 (Pin_6)
- net A7: now also J3.4 (Pin_4); no longer J3.5 (Pin_5)
- net A8: now also J3.3 (Pin_3); no longer J3.4 (Pin_4)
- net A9: now also J3.2 (Pin_2); no longer J3.3 (Pin_3)
- net CLK: now also J2.6 (Pin_6); no longer J2.7 (Pin_7)
- net D0: now also J2.14 (Pin_14); no longer J2.15 (Pin_15)
- net D1: now also J2.15 (Pin_15); no longer J2.16 (Pin_16)
- net D2: now also J2.12 (Pin_12); no longer J2.13 (Pin_13)
- net D3: now also J2.8 (Pin_8); no longer J2.9 (Pin_9)
- net D4: now also J2.7 (Pin_7); no longer J2.8 (Pin_8)
- net D5: now also J2.9 (Pin_9); no longer J2.10 (Pin_10)
- net D6: now also J2.10 (Pin_10); no longer J2.11 (Pin_11)
- net D7: now also J2.13 (Pin_13); no longer J2.14 (Pin_14)
- net GND: now also J3.12 (Pin_12); no longer J3.13 (Pin_13)
- net VCC: now also J2.11 (Pin_11); no longer J2.12 (Pin_12)
- net ~{BUSAK}: now also J3.18 (Pin_18); no longer J3.19 (Pin_19)
- net ~{BUSRQ}: now also J3.16 (Pin_16); no longer J3.17 (Pin_17)
- net ~{INT}: now also J2.16 (Pin_16); no longer J2.17 (Pin_17)
- net ~{IORQ}: now also J2.20 (Pin_20); no longer J2.21 (Pin_21)
- net ~{M1}: now also J3.14 (Pin_14); no longer J3.15 (Pin_15)
- net ~{MREQ}: now also J2.19 (Pin_19); no longer J2.20 (Pin_20)
- net ~{NMI}: now also J2.17 (Pin_17); no longer J2.18 (Pin_18)
- net ~{RD}: now also J3.20 (Pin_20); no longer J3.21 (Pin_21)
- net ~{ROM_WE}: now also J3.21 (Pin_21); no longer J3.1 (Pin_1)
- net ~{RST}: now also J3.15 (Pin_15); no longer J3.16 (Pin_16)
- net ~{WR}: now also J3.19 (Pin_19); no longer J3.20 (Pin_20)
Other:
- added sheet Debugger (debugger.kicad_sch)
- moved on the sheet: J2, J3
