File: fortuna-s/fortuna-s.kicad_sch (KiCad schematic)
At the start: 42 parts, among them J1 Ext Pinout, J2 Conn_01x21, J3 Conn_01x21, U1 74HTC138, U2 74HTC175

Commit message: .
Parts:
- added JP1: Clock, symbol Jumper:Jumper_2_Open
Connections:
- net ~{RST}: now also JP1.2 (B); no longer C?.1, D?.2 (A), R?.1, R?.1
- new net: C?.1, D?.2 (A), JP1.1 (A), R?.1, R?.1
Changed lines of the file:
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@@
     (stroke (width 0) (type default))
   )
-  (wire (pts (xy 105.41 130.81) (xy 119.38 130.81))
+  (wire (pts (xy 105.41 130.81) (xy 111.125 130.81))
     (stroke (width 0) (type default))
   )
@@
   )
   (wire (pts (xy 99.06 153.67) (xy 99.06 156.21))
+    (stroke (width 0) (type default))
+  )
+  (wire (pts (xy 121.285 130.81) (xy 129.54 130.81))
     (stroke (width 0) (type default))
   )
@@
     (effects (font (size 1.27 1.27)) (justify left bottom))
   )
+  (label "~{RST}" (at 129.54 130.81 180) (fields_autoplaced)
+    (effects (font (size 1.27 1.27)) (justify right bottom))
+  )
   (label "~{IORQ}" (at 162.56 226.695 0) (fields_autoplaced)
     (effects (font (size 1.27 1.27)) (justify left bottom))
@@
   )
   (label "~{Y3R}" (at 389.89 210.82 180) (fields_autoplaced)
-    (effects (font (size 1.27 1.27)) (justify right bottom))
-  )
-  (label "~{RST}" (at 119.38 130.81 180) (fields_autoplaced)
     (effects (font (size 1.27 1.27)) (justify right bottom))
   )
@@
         )
       )
+    )
+  )
+  (symbol (lib_id "Jumper:Jumper_2_Open") (at 116.205 130.81 0) (unit 1)
+    (in_bom yes) (on_board yes) (dnp no) (fields_autoplaced)
+    (property "Reference" "JP1" (at 116.205 124.46 0)
+      (effects (font (size 1.27 1.27)))
+    )
+    (property "Value" "Clock" (at 116.205 127 0)
+      (effects (font (size 1.27 1.27)))
+    )
+    (property "Footprint" "" (at 116.205 130.81 0)
+      (effects (font (size 1.27 1.27)) hide)
+    )
+    (property "Datasheet" "~" (at 116.205 130.81 0)
+      (effects (font (size 1.27 1.27)) hide)
+    )
+    (pin "1")
+    (pin "2")
+    (instances
+      (project "fortuna-s"
+        (path "/01925f6f-51ef-4838-b51d-68dc0814d806"
+          (reference "JP1") (unit 1)
+        )
+      )

Commit message: .
Parts:
- added J6: Power (to panel), symbol Connector_Generic:Conn_02x01
Connections:
- net GND: now also J6.1 (Pin_1)
- net VCC: now also J6.2 (Pin_2)
Other:
- moved on the sheet: D?, R?
Changed lines of the file:
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@@
     (stroke (width 0) (type default))
   )
-  (wire (pts (xy 88.9 44.45) (xy 88.9 49.53))
+  (wire (pts (xy 83.82 44.45) (xy 83.82 49.53))
     (stroke (width 0) (type default))
   )
@@
     (stroke (width 0) (type default))
   )
-  (wire (pts (xy 68.58 44.45) (xy 88.9 44.45))
+  (wire (pts (xy 68.58 44.45) (xy 83.82 44.45))
     (stroke (width 0) (type default))
   )
@@
     (stroke (width 0) (type default))
   )
-  (wire (pts (xy 88.9 66.04) (xy 88.9 67.31))
+  (wire (pts (xy 83.82 66.04) (xy 83.82 67.31))
     (stroke (width 0) (type default))
   )
@@
     (stroke (width 0) (type default))
   )
-  (wire (pts (xy 88.9 57.15) (xy 88.9 58.42))
+  (wire (pts (xy 83.82 57.15) (xy 83.82 58.42))
     (stroke (width 0) (type default))
   )
@@
     )
   )
-  (symbol (lib_id "Device:R_US") (at 88.9 62.23 0) (unit 1)
+  (symbol (lib_id "Device:R_US") (at 83.82 62.23 0) (unit 1)
     (in_bom yes) (on_board yes) (dnp no)
-    (property "Reference" "R?" (at 91.44 60.9599 0)
+    (property "Reference" "R?" (at 86.36 60.9599 0)
       (effects (font (size 1.27 1.27)) (justify left))
     )
-    (property "Value" "100" (at 91.44 63.4999 0)
+    (property "Value" "100" (at 86.36 63.4999 0)
       (effects (font (size 1.27 1.27)) (justify left))
     )
-    (property "Footprint" "" (at 89.916 62.484 90)
+    (property "Footprint" "" (at 84.836 62.484 90)
       (effects (font (size 1.27 1.27)) hide)
     )
-    (property "Datasheet" "~" (at 88.9 62.23 0)
+    (property "Datasheet" "~" (at 83.82 62.23 0)
       (effects (font (size 1.27 1.27)) hide)
     )
@@
     )
   )
+  (symbol (lib_id "power:VCC") (at 100.965 48.895 0) (unit 1)
+    (in_bom yes) (on_board yes) (dnp no) (fields_autoplaced)
+    (property "Reference" "#PWR017" (at 100.965 52.705 0)
+      (effects (font (size 1.27 1.27)) hide)
+    )
+    (property "Value" "VCC" (at 100.965 43.815 0)
+      (effects (font (size 1.27 1.27)))
+    )
+    (property "Footprint" "" (at 100.965 48.895 0)
+      (effects (font (size 1.27 1.27)) hide)
+    )
+    (property "Datasheet" "" (at 100.965 48.895 0)
+      (effects (font (size 1.27 1.27)) hide)
+    )
+    (pin "1")
+    (instances
+      (project "fortuna-s"
+        (path "/01925f6f-51ef-4838-b51d-68dc0814d806"
+          (reference "#PWR017") (unit 1)
+        )
+      )
+    )
+  )
   (symbol (lib_id "Jumper:Jumper_2_Open") (at 116.205 130.81 0) (unit 1)
     (in_bom yes) (on_board yes) (dnp no) (fields_autoplaced)
@@
     )
   )
-  (symbol (lib_id "Device:LED") (at 88.9 53.34 90) (unit 1)
+  (symbol (lib_id "Device:LED") (at 83.82 53.34 90) (unit 1)
     (in_bom yes) (on_board yes) (dnp no) (fields_autoplaced)
-    (property "Reference" "D?" (at 92.71 53.6574 90)
+    (property "Reference" "D?" (at 87.63 53.6574 90)
       (effects (font (size 1.27 1.27)) (justify right))
     )
-    (property "Value" "GREEN" (at 92.71 56.1974 90)
+    (property "Value" "GREEN" (at 87.63 56.1974 90)
       (effects (font (size 1.27 1.27)) (justify right))
     )
-    (property "Footprint" "" (at 88.9 53.34 0)
+    (property "Footprint" "" (at 83.82 53.34 0)
       (effects (font (size 1.27 1.27)) hide)
     )
-    (property "Datasheet" "~" (at 88.9 53.34 0)
+    (property "Datasheet" "~" (at 83.82 53.34 0)
       (effects (font (size 1.27 1.27)) hide)
     )
@@
     )
   )
+  (symbol (lib_id "Connector_Generic:Conn_02x01") (at 100.965 56.515 90) (unit 1)
+    (in_bom yes) (on_board yes) (dnp no)
+    (property "Reference" "J6" (at 103.505 53.975 90)
+      (effects (font (size 1.27 1.27)) (justify right))
+    )
+    (property "Value" "Power (to panel)" (at 103.505 56.515 90)
+      (effects (font (size 1.27 1.27)) (justify right))
+    )
+    (property "Footprint" "" (at 100.965 56.515 0)
+      (effects (font (size 1.27 1.27)) hide)
+    )
+    (property "Datasheet" "~" (at 100.965 56.515 0)
+      (effects (font (size 1.27 1.27)) hide)
+    )
+    (pin "1")
+    (pin "2")
+    (instances
+      (project "fortuna-s"
+        (path "/01925f6f-51ef-4838-b51d-68dc0814d806"
+          (reference "J6") (unit 1)
+        )
+      )
+    )
+  )
   (symbol (lib_id "74xx:74HCT04") (at 316.23 92.71 0) (unit 1)
     (in_bom yes) (on_board yes) (dnp no)
@@
     )
   )
+  (symbol (lib_id "power:GND") (at 100.965 61.595 0) (unit 1)
+    (in_bom yes) (on_board yes) (dnp no) (fields_autoplaced)
+    (property "Reference" "#PWR018" (at 100.965 67.945 0)
+      (effects (font (size 1.27 1.27)) hide)
+    )
+    (property "Value" "GND" (at 100.965 66.675 0)
+      (effects (font (size 1.27 1.27)))
+    )
+    (property "Footprint" "" (at 100.965 61.595 0)
+      (effects (font (size 1.27 1.27)) hide)
+    )
+    (property "Datasheet" "" (at 100.965 61.595 0)
+      (effects (font (size 1.27 1.27)) hide)
+    )
+    (pin "1")
+    (instances
+      (project "fortuna-s"
+        (path "/01925f6f-51ef-4838-b51d-68dc0814d806"
+          (reference "#PWR018") (unit 1)
+        )
+      )
+    )
+  )
   (symbol (lib_id "power:VCC") (at 367.03 49.53 0) (unit 1)
     (in_bom yes) (on_board yes) (dnp no) (fields_autoplaced)
@@
     )
   )
-  (symbol (lib_id "power:GND") (at 88.9 67.31 0) (unit 1)
+  (symbol (lib_id "power:GND") (at 83.82 67.31 0) (unit 1)
     (in_bom yes) (on_board yes) (dnp no) (fields_autoplaced)
-    (property "Reference" "#PWR?" (at 88.9 73.66 0)
+    (property "Reference" "#PWR?" (at 83.82 73.66 0)
       (effects (font (size 1.27 1.27)) hide)
     )
-    (property "Value" "GND" (at 88.9 72.39 0)
+    (property "Value" "GND" (at 83.82 72.39 0)
       (effects (font (size 1.27 1.27)))
     )
-    (property "Footprint" "" (at 88.9 67.31 0)
+    (property "Footprint" "" (at 83.82 67.31 0)
       (effects (font (size 1.27 1.27)) hide)
     )
-    (property "Datasheet" "" (at 88.9 67.31 0)
+    (property "Datasheet" "" (at 83.82 67.31 0)
       (effects (font (size 1.27 1.27)) hide)
     )

Commit message: .
Other:
- note added: "Board design"
- moved on the sheet: C1, C2, C?, J1, J2, J3, U1, U2

Commit message: .
Connections:
- net CLK: no longer U?.3 (Rx_CLK), U?.4 (Tx_CLK)
- net CLK_UART: now reaches JP?.1 (A), X?.8 (OUT)
- net CLK_UART: now also U?.3 (Rx_CLK), U?.4 (Tx_CLK)
Changed lines of the file:
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@@
   (junction (at 226.06 92.71) (diameter 0) (color 0 0 0 0)
+  )
+  (junction (at 52.07 127) (diameter 0) (color 0 0 0 0)
   )
   (junction (at 36.83 215.9) (diameter 0) (color 0 0 0 0)
@@
     (stroke (width 0) (type default))
   )
-  (wire (pts (xy 330.2 100.33) (xy 335.28 100.33))
+  (wire (pts (xy 323.85 100.33) (xy 335.28 100.33))
     (stroke (width 0) (type default))
   )
@@
     (stroke (width 0) (type default))
   )
+  (wire (pts (xy 52.07 127) (xy 52.07 133.35))
+    (stroke (width 0) (type default))
+  )
   (wire (pts (xy 340.995 187.96) (xy 334.645 187.96))
     (stroke (width 0) (type default))
@@
     (stroke (width 0) (type default))
   )
-  (wire (pts (xy 49.53 127) (xy 54.61 127))
+  (wire (pts (xy 49.53 127) (xy 52.07 127))
     (stroke (width 0) (type default))
   )
@@
     (stroke (width 0) (type default))
   )
+  (wire (pts (xy 52.07 133.35) (xy 71.12 133.35))
+    (stroke (width 0) (type default))
+  )
   (wire (pts (xy 380.365 176.53) (xy 389.255 176.53))
     (stroke (width 0) (type default))
@@
   )
   (wire (pts (xy 234.315 175.26) (xy 245.745 175.26))
+    (stroke (width 0) (type default))
+  )
+  (wire (pts (xy 52.07 127) (xy 54.61 127))
     (stroke (width 0) (type default))
   )
@@
     (effects (font (size 1.27 1.27)) (justify left bottom))
   )
-  (label "CLK" (at 330.2 100.33 0) (fields_autoplaced)
+  (label "CLK_UART" (at 323.85 100.33 0) (fields_autoplaced)
     (effects (font (size 1.27 1.27)) (justify left bottom))
   )
@@
     (effects (font (size 1.27 1.27)) (justify left bottom))
   )
+  (label "CLK_UART" (at 71.12 133.35 180) (fields_autoplaced)
+    (effects (font (size 1.27 1.27)) (justify right bottom))
+  )
   (label "~{RST}" (at 53.34 200.66 0) (fields_autoplaced)

Commit message: .
Connections:
- net VCC: now also P?.A4 (VBUS), P?.A9 (VBUS), P?.B4 (VBUS), P?.B9 (VBUS), SW?.1; no longer SW?.2, SW?.3
Other:
- moved on the sheet: D?, J6, R?

Commit message: .
Parts:
- removed C1, C2, C? (x4): 10uF, symbol Device:C
- removed J1: Ext Pinout, symbol Connector_Generic:Conn_02x13_Counter_Clockwise
- removed J2, J3: Conn_01x21, symbol Connector_Generic:Conn_01x21
- removed J?: FTDI cable, symbol Connector_Generic:Conn_01x06
- removed R? (x4): 10K, symbol Device:R_US
- removed R?: 3k3, symbol Device:R_US
- removed U1: 74HTC138, symbol 74xx:74LS138
- removed U2: 74HTC175, symbol 74xx:74LS175
- removed U? (x4): 74LS32, symbol 74xx:74LS32
- removed U?: 28C256, symbol Memory_EEPROM:28C256
- removed U?: AS6C4008-55PCN, Package_DIP:DIP-32_W15.24mm, symbol Memory_RAM:AS6C4008-55PCN
- removed U?: MC68B50, Package_DIP:DIP-40_W15.24mm, symbol Interface_UART:MC68B50
- removed U? (x2): 74HCT04, symbol 74xx:74HCT04
Connections:
- net VCC: no longer P?.A4 (VBUS), P?.A9 (VBUS), P?.B4 (VBUS), P?.B9 (VBUS), SW?.1
- net CLK_UART renamed CLK_EXT
- new net 5V_FTDI: P?.A4 (VBUS), P?.A9 (VBUS), P?.B4 (VBUS), P?.B9 (VBUS), SW?.1
- no-connect marks 18 -> 7
Other:
- added sheet Memory (memory.kicad_sch)
- added sheet Peripheral (peripheral.kicad_sch)
- note removed: "0x80 - Write serial 0x81 - Read serial"
- note removed: "BANKSWITCHING"
- note removed: "DEBUGGER"
- note removed: "EXTERNAL I/O"
- note removed: "I/O MULTIPLEXER"
- note removed: "IO address: write to 0x0"
- note removed: "MEMORY"
- note removed: "Occupies 0x80 to 0xBF in memory map."
- note removed: "The computer can be powered by the FTDI cable, but current can't exceed 350 mA."
- note removed: "UART"
- note removed: "UART communcates at 115000 baud."
- moved on the sheet: C?, D?, J6, JP1, JP?, P?, R?, SW?, U?, X?

Commit message: .
Parts:
- added U1: 74HTC138, symbol 74xx:74LS138
Connections:
- net GND: now also U1.8 (GND)
- net VCC: now also U1.16 (VCC)
- net ~{IORQ}: now also U1.5 (E2)
- net ~{M1}: now also U1.6 (E3)
- new net A0: U1.2 (A1)
- new net A1: U1.3 (A2)
- new net A7: U1.4 (E1)
- new net WR: U1.1 (A0)
- new net ~{Y0R}: U1.14 (O1)
- new net ~{Y0W}: U1.15 (O0)
- new net ~{Y1R}: U1.12 (O3)
- new net ~{Y1W}: U1.13 (O2)
- new net ~{Y2R}: U1.10 (O5)
- new net ~{Y2W}: U1.11 (O4)
- new net ~{Y3R}: U1.7 (O7)
- new net ~{Y3W}: U1.9 (O6)
Other:
- note added: "I/O MULTIPLEXER"
- moved on the sheet: C?, D?, JP1, JP?, R?, SW?, X?

Commit message: .
Changed lines of the file:
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@@
     (stroke (width 0) (type default))
   )
-  (rectangle (start 25.4 146.685) (end 118.11 193.675)
+  (rectangle (start 25.4 146.685) (end 116.205 193.675)
     (stroke (width 0.3) (type default))
     (fill (type none))
@@
   )
   (text_box "ATMega8\n(SDCard)"
-    (at 100.33 171.45 0) (size 10.16 21.59)
+    (at 81.915 172.085 0) (size 8.255 19.685)
     (stroke (width 0) (type default))
     (fill (type none))
@@
   )
   (text_box "SDCard"
-    (at 82.55 173.99 0) (size 12.7 20.32)
+    (at 92.075 172.085 0) (size 12.7 21.59)
     (stroke (width 0) (type default))
     (fill (type none))
@@
   )
   (text_box "74HCT138\n(demux)"
-    (at 71.12 168.91 0) (size 8.89 10.16)
+    (at 70.485 168.91 0) (size 8.89 10.16)
     (stroke (width 0) (type default))
     (fill (type none))
@@
   )
   (text_box "VGA\nadaptor"
-    (at 100.33 146.05 0) (size 17.78 13.97)
+    (at 99.06 146.05 0) (size 17.78 13.97)
     (stroke (width 0) (type default))
     (fill (type none))
@@
   )
   (text_box "LED"
-    (at 96.52 184.15 0) (size 2.54 8.89)
+    (at 106.045 184.785 0) (size 2.54 8.89)
     (stroke (width 0) (type default))
     (fill (type none))
@@
   )
   (text_box "PI Pico\n(VGA)"
-    (at 83.82 146.05 0) (size 12.7 25.4)
+    (at 83.82 146.05 0) (size 12.7 24.765)
     (stroke (width 0) (type default))
     (fill (type none))
@@
   )
   (text_box "74HC74\n(flipflop)"
-    (at 71.12 181.61 0) (size 8.89 10.16)
+    (at 70.485 181.61 0) (size 8.89 10.16)
     (stroke (width 0) (type default))
     (fill (type none))
