File: fortuna-s/debugger.kicad_sch (KiCad schematic)
At the start: 3 parts, among them J2 Conn_01x21, J3 Conn_01x21

Commit message: .
Connections:
- net A10: now also XA1.A8; no longer XA1.A0
- net A6: now also XA1.A0; no longer XA1.A8
- net A7: now also XA1.A2; no longer XA1.A6
- net A9: now also XA1.A6; no longer XA1.A2
