File: fortuna-s/memory.kicad_sch (KiCad schematic)
At the start: 18 parts, among them U2 74HTC175

Commit message: .
Parts:
- added U?: 74HCT04, symbol 74xx:74HCT04
Connections:
- net ~{Y0W}: now also U?.9; no longer U2.9 (Cp)
- new net: U2.9 (Cp), U?.8
Changed lines of the file:
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@@
+    (stroke (width 0) (type default))
+  )
+  (wire (pts (xy 180.975 77.47) (xy 187.96 77.47))
     (stroke (width 0) (type default))
   )
@@
     (effects (font (size 1.27 1.27)) (justify left bottom))
   )
+  (label "~{Y0W}" (at 180.975 77.47 0) (fields_autoplaced)
+    (effects (font (size 1.27 1.27)) (justify left bottom))
+  )
   (label "ADDR" (at 45.72 49.53 0) (fields_autoplaced)
     (effects (font (size 1.27 1.27)) (justify left bottom))
@@
   )
   (label "D1" (at 203.2 62.23 0) (fields_autoplaced)
-    (effects (font (size 1.27 1.27)) (justify left bottom))
-  )
-  (label "~{Y0W}" (at 203.2 77.47 0) (fields_autoplaced)
     (effects (font (size 1.27 1.27)) (justify left bottom))
   )
@@
         )
       )
+    )
+  )
+  (symbol (lib_id "74xx:74HCT04") (at 195.58 77.47 0) (unit 4)
+    (in_bom yes) (on_board yes) (dnp no) (fields_autoplaced)
+    (property "Reference" "U?" (at 195.58 69.215 0)
+      (effects (font (size 1.27 1.27)))
+    )
+    (property "Value" "74HCT04" (at 195.58 71.755 0)
+      (effects (font (size 1.27 1.27)))
+    )
+    (property "Footprint" "" (at 195.58 77.47 0)
+      (effects (font (size 1.27 1.27)) hide)
+    )
+    (property "Datasheet" "https://assets.nexperia.com/documents/data-sheet/74HC_HCT04.pdf" (at 195.58 77.47 0)
+      (effects (font (size 1.27 1.27)) hide)
+    )
+    (pin "1")
+    (pin "2")
+    (pin "3")
+    (pin "4")
+    (pin "5")
+    (pin "6")
+    (pin "8")
+    (pin "9")
+    (pin "10")
+    (pin "11")
+    (pin "12")
+    (pin "13")
+    (pin "14")
+    (pin "7")
+    (instances
+      (project "fortuna-s"
+        (path "/01925f6f-51ef-4838-b51d-68dc0814d806"
+          (reference "U?") (unit 4)
+        )
+        (path "/01925f6f-51ef-4838-b51d-68dc0814d806/d4082d08-879a-4830-8eba-96c650883a9b"
+          (reference "U10") (unit 2)
+        )
+      )
